File: hardware/if_amp.sch (KiCad schematic (older format))
At the start: 106 parts, among them Q301 2N3904, Q302 2N3904, Q303 2N3904, Q304 2N3904, Q305 2N3904, Q306 2N3904, Q307 2N3904, Q308 2N3904, Q309 2N3904, Q310 2N3904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

Commit message: initial commit
Connections:
- net GND: now also T301.3 (SA); no longer T301.4 (SB)
- net at Q310.2 (B), R329.1: now also T301.4 (SB); no longer T301.3 (SA)
Changed lines of the file:
@@
 Wire Wire Line
 	13600 4000 13600 4300
-Wire Wire Line
-	13050 4400 13300 4400
-Wire Wire Line
-	13300 4400 13300 4000
-Wire Wire Line
-	13300 4000 13600 4000
 Connection ~ 13600 4000
-$Comp
-L power:GND #PWR0329
-U 1 1 5FA99B95
-P 13050 4000
-F 0 "#PWR0329" H 13050 3750 50  0001 C CNN
-F 1 "GND" H 13055 3827 50  0000 C CNN
-F 2 "" H 13050 4000 50  0001 C CNN
-F 3 "" H 13050 4000 50  0001 C CNN
-	1    13050 4000
-	1    0    0    -1
-$EndComp
 Wire Wire Line
 	15550 4000 15550 6150
@@
 Text Notes 12525 3725 0    50   ~ 0
 FT37-43
+$Comp
+L power:GND #PWR?
+U 1 1 5FD106B6
+P 13050 4400
+F 0 "#PWR?" H 13050 4150 50  0001 C CNN
+F 1 "GND" H 13055 4227 50  0000 C CNN
+F 2 "" H 13050 4400 50  0001 C CNN
+F 3 "" H 13050 4400 50  0001 C CNN
+	1    13050 4400
+	1    0    0    -1
+$EndComp
+Wire Wire Line
+	13050 4000 13600 4000
 $EndSCHEMATC
